File: EAGLE/projects/IDP/IDP5.brd (EAGLE design)
At the start: 100 x 80 mm, 13 parts, among them M1 IDP_PROTOBOARD

Commit message: Ready for submission
Parts:
- LED1, LED2, LED3: value LED_23MM -> 55-1776
- PHOTO: value 22-05-7028-02 -> Rapid 22-0905/22-1005
Changed lines of the file:
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@@
 <attribute name="VALUE" x="47.809609375" y="26.60221875" size="1.273109375" layer="27" rot="R270"/>
 </element>
-<element name="PHOTO" library="IDP_library" package="7395-02" package3d_urn="urn:adsk.eagle:package:8078644/1" value="22-05-7028-02" x="35.56" y="19.05" smashed="yes">
+<element name="PHOTO" library="IDP_library" package="7395-02" package3d_urn="urn:adsk.eagle:package:8078644/1" value="Rapid 22-0905/22-1005" x="35.56" y="19.05" smashed="yes">
 <attribute name="MF" value="MOLEX" x="35.56" y="19.05" size="1.778" layer="27" display="off"/>
 <attribute name="MPN" value="" x="35.56" y="19.05" size="1.778" layer="27" display="off"/>
@@
 <attribute name="VALUE" x="35.1521" y="25.5001" size="0.8128" layer="27" ratio="10" rot="R270"/>
 </element>
-<element name="LED2" library="IDP_library" package="LED3MM" package3d_urn="urn:adsk.eagle:package:15797/1" value="LED_23MM" x="67.31" y="49.53" smashed="yes" rot="R270">
+<element name="LED2" library="IDP_library" package="LED3MM" package3d_urn="urn:adsk.eagle:package:15797/1" value="55-1776" x="67.31" y="49.53" smashed="yes" rot="R270">
 <attribute name="NAME" x="60.325" y="47.371" size="1.27" layer="25" ratio="10"/>
 <attribute name="POPULARITY" value="97" x="67.31" y="49.53" size="1.778" layer="27" rot="R270" display="off"/>
 </element>
-<element name="LED3" library="IDP_library" package="LED3MM" package3d_urn="urn:adsk.eagle:package:15797/1" value="LED_23MM" x="69.85" y="44.45" smashed="yes" rot="R270">
+<element name="LED3" library="IDP_library" package="LED3MM" package3d_urn="urn:adsk.eagle:package:15797/1" value="55-1776" x="69.85" y="44.45" smashed="yes" rot="R270">
 <attribute name="NAME" x="71.755" y="42.291" size="1.27" layer="25" ratio="10"/>
 <attribute name="POPULARITY" value="97" x="69.85" y="44.45" size="1.778" layer="27" rot="R270" display="off"/>
@@
 <attribute name="VALUE" x="64.897" y="32.512" size="1.27" layer="27" ratio="10" rot="R90"/>
 </element>
-<element name="LED1" library="IDP_library" package="LED3MM" package3d_urn="urn:adsk.eagle:package:15797/1" value="LED_23MM" x="36.83" y="30.48" smashed="yes" rot="R90">
+<element name="LED1" library="IDP_library" package="LED3MM" package3d_urn="urn:adsk.eagle:package:15797/1" value="55-1776" x="36.83" y="30.48" smashed="yes" rot="R90">
 <attribute name="NAME" x="36.449" y="32.385" size="1.27" layer="25" ratio="10" rot="R90"/>
 <attribute name="POPULARITY" value="97" x="36.83" y="30.48" size="1.778" layer="27" rot="R90" display="off"/>

Commit message: Final Version
Parts:
- added LED4: 55-1776, IDP_library:LED3MM
- added PHOTO1: Rapid 22-0905/22-1005, IDP_library:7395-02
- added RAPID65-0001: 5K, IDP_library:TRIM_3296W-1-250
Connections:
- new net PHOTO_ALALOG1: LED4.A, PHOTO1.1, RAPID65-0001.3
- new net PHOTO_ANALOG_2: LED4.K, M1.A5
- net +5V: now also PHOTO1.2
- net GND: now also RAPID65-0001.1
Routing:
- net PHOTO_ANALOG_2: track 0.00 -> 72.4 mm, vias 0 -> 2
- net +5V: track 43.2 -> 59.7 mm, vias 0 -> 2
- net PHOTO_ALALOG1: track 0.00 -> 10.2 mm
- net GND: track 69.9 -> 77.5 mm
Changed lines of the file:
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@@
 <attribute name="VALUE" x="38.481" y="32.385" size="1.27" layer="27" ratio="10" rot="R90"/>
+</element>
+<element name="RAPID65-0001" library="IDP_library" package="TRIM_3296W-1-250" value="5K" x="24.13" y="22.86" smashed="yes" rot="R180">
+<attribute name="AVAILABILITY" value="Unavailable" x="24.13" y="3.81" size="1.778" layer="27" rot="R180" display="off"/>
+<attribute name="DESCRIPTION" value=" Trimpot 25 Ohm 3/8 Sq Cer Mt " x="24.13" y="3.81" size="1.778" layer="27" rot="R180" display="off"/>
+<attribute name="MF" value="Bourns" x="24.13" y="3.81" size="1.778" layer="27" rot="R180" display="off"/>
+<attribute name="MP" value="3296W-1-250" x="24.13" y="3.81" size="1.778" layer="27" rot="R180" display="off"/>
+<attribute name="NAME" x="29.151440625" y="19.847140625" size="1.275440625" layer="25" rot="R180"/>
+<attribute name="PACKAGE" value="SOT-23-5 Bourns" x="24.13" y="3.81" size="1.778" layer="27" rot="R180" display="off"/>
+<attribute name="PRICE" value="None" x="24.13" y="3.81" size="1.778" layer="27" rot="R180" display="off"/>
+<attribute name="VALUE" x="29.14221875" y="27.120390625" size="1.273109375" layer="27" rot="R180"/>
+</element>
+<element name="PHOTO1" library="IDP_library" package="7395-02" package3d_urn="urn:adsk.eagle:package:8078644/1" value="Rapid 22-0905/22-1005" x="15.24" y="24.13" smashed="yes" rot="R270">
+<attribute name="MF" value="MOLEX" x="24.13" y="33.02" size="1.778" layer="27" rot="R270" display="off"/>
+<attribute name="MPN" value="" x="24.13" y="33.02" size="1.778" layer="27" rot="R270" display="off"/>
+<attribute name="NAME" x="13.1079" y="29.1099" size="1.016" layer="25" ratio="10" rot="R90"/>
+<attribute name="OC_FARNELL" value="9731601" x="24.13" y="33.02" size="1.778" layer="27" rot="R270" display="off"/>
+<attribute name="OC_NEWARK" value="unknown" x="24.13" y="33.02" size="1.778" layer="27" rot="R270" display="off"/>
+<attribute name="POPULARITY" value="0" x="24.13" y="33.02" size="1.778" layer="27" rot="R270" display="off"/>
+<attribute name="VALUE" x="13.5621" y="39.4701" size="0.8128" layer="27" ratio="10" rot="R270"/>
+</element>
+<element name="LED4" library="IDP_library" package="LED3MM" package3d_urn="urn:adsk.eagle:package:15797/1" value="55-1776" x="21.59" y="27.94" smashed="yes" rot="R90">
+<attribute name="NAME" x="21.209" y="31.115" size="1.27" layer="25" ratio="10" rot="R90"/>
+<attribute name="POPULARITY" value="97" x="2.54" y="19.05" size="1.778" layer="27" rot="R90" display="off"/>
+<attribute name="VALUE" x="23.241" y="29.845" size="1.27" layer="27" ratio="10" rot="R90"/>
 </element>
 </elements>
@@
 <wire x1="59.69" y1="35.56" x2="62.23" y2="35.56" width="0.1524" layer="1"/>
 <wire x1="44.45" y1="25.4" x2="44.45" y2="20.32" width="0.1524" layer="16"/>
+<contactref element="RAPID65-0001" pad="1"/>
+<wire x1="26.67" y1="22.86" x2="26.67" y2="15.24" width="0.1524" layer="16"/>
 <wire x1="59.69" y1="20.32" x2="59.69" y2="22.86" width="0" layer="19" extent="16-16"/>
 </signal>
@@
 <wire x1="57.15" y1="29.21" x2="57.15" y2="22.86" width="0.1524" layer="16"/>
 <wire x1="34.29" y1="38.1" x2="34.29" y2="19.05" width="0.1524" layer="16"/>
+<contactref element="PHOTO1" pad="2"/>
+<via x="19.05" y="25.4" extent="1-16" drill="0.35"/>
+<via x="19.05" y="38.1" extent="1-16" drill="0.35"/>
+<wire x1="19.05" y1="38.1" x2="19.05" y2="25.4" width="0.1524" layer="1"/>
+<wire x1="15.24" y1="25.4" x2="19.05" y2="25.4" width="0.1524" layer="1"/>
 </signal>
 <signal name="MOTOR_CHANNEL_A_DIRECTION">
@@
 <via x="69.85" y="17.78" extent="1-16" drill="0.35"/>
 </signal>
+<signal name="PHOTO_ALALOG1">
+<contactref element="PHOTO1" pad="1"/>
+<contactref element="RAPID65-0001" pad="3"/>
+<contactref element="LED4" pad="A"/>
+<wire x1="15.24" y1="22.86" x2="21.59" y2="22.86" width="0.1524" layer="1"/>
+<wire x1="21.59" y1="26.67" x2="21.59" y2="22.86" width="0.1524" layer="16"/>
+</signal>
+<signal name="PHOTO_ANALOG_2">
+<contactref element="LED4" pad="K"/>
+<contactref element="M1" pad="A5"/>
+<via x="31.75" y="29.21" extent="1-16" drill="0.35"/>
+<wire x1="21.59" y1="29.21" x2="31.75" y2="29.21" width="0.1524" layer="1"/>
+<wire x1="31.75" y1="29.21" x2="31.75" y2="13.97" width="0.1524" layer="1"/>
+<wire x1="31.75" y1="13.97" x2="74.93" y2="13.97" width="0.1524" layer="1"/>
+<wire x1="74.93" y1="13.97" x2="74.93" y2="17.78" width="0.1524" layer="1"/>
+<via x="74.93" y="17.78" extent="1-16" drill="0.35"/>
+</signal>
 </signals>

Commit message: few changes
Parts:
- removed LED4: 55-1776, IDP_library:LED3MM
- moved LED1 40.3 mm to (72.4, 49.5), turned to 270 degrees
- moved PHOTO1 2.84 mm to (14.0, 26.7)
- moved RAPID65-0001 2.54 mm to (21.6, 22.9), turned to 90 degrees
- moved RAPID65-0753 2.54 mm to (39.4, 25.4)
Connections:
- removed net PHOTO_ALALOG: LED1.A, PHOTO.1, RAPID65-0753.3
- removed net PHOTO_ALALOG1: LED4.A, PHOTO1.1, RAPID65-0001.3
- new net COLOUR_CONFIRM: LED1.A, M1.D1
- net GND: now also LED1.K
- net PHOTO_ANALOG: now also PHOTO.1, RAPID65-0753.3; no longer LED1.K
- net PHOTO_ANALOG_2: now also PHOTO1.1, RAPID65-0001.3; no longer LED4.K
Routing:
- net PHOTO_ANALOG: track 57.1 -> 41.9 mm, vias 3 -> 2
- net PHOTO_ALALOG: track 12.7 -> 0.00 mm, vias 1 -> 0
- net COLOUR_CONFIRM: track 0.00 -> 10.2 mm, vias 0 -> 2
- net PHOTO_ALALOG1: track 10.2 -> 0.00 mm
- net GND: track 77.5 -> 82.6 mm
- net +5V: track 59.7 -> 55.9 mm, vias 2 -> 3
- net PHOTO_ANALOG_2: track 72.4 -> 76.2 mm
